File: HVAC/UnderfloorHeating/UnderfloorHeatingActuatorsControl/220V/uhc-12/io220v.kicad_sch (KiCad schematic)
At the start: 4 parts, among them Q1 MAC97A8

Commit message: Reorganization
Parts:
- removed Q1: MAC97A8, Digikey:SOT-23-3, symbol PCM_Triac_AKL:MAC97A8
- removed R?: 300/1w, Resistor_SMD:R_2512_6332Metric, symbol Device:R
- removed R?: 91, Resistor_SMD:R_0805_2012Metric_Pad1.20x1.40mm_HandSolder, symbol Device:R
- added Q11: BT137S-800F, Package_TO_SOT_SMD_AKL:TO-252-2, symbol PCM_Triac_AKL:BT137S-800F
- added R?: 91, Resistor_SMD:R_0805_2012Metric_Pad1.20x1.40mm_HandSolder, symbol Device:R
- added R?: 300/1w, Resistor_SMD:R_2512_6332Metric, symbol Device:R
Connections:
- net 220V_out: now also Q11.1 (A1)
- net 220_IN: now also Q11.2 (A2), R?.2
- net Control: now also R?.1
- net at OC1.1: now also R?.2
- net at OC1.4: now also Q11.3 (G)
- net at OC1.6: now also R?.1
