File: HVAC/UnderfloorHeating/UnderfloorHeatingActuatorsControl/220V/uhc-12/power_sch.kicad_sch (KiCad schematic)
At the start: 11 parts, among them J7 220IN, U2 LM3671MFX-3.3/NOPB

Commit message: Reorganization
Parts:
- removed J7: 220IN, Connector_JST:JST_NV_B02P-NV_1x02_P5.00mm_Vertical, symbol Connector:Conn_01x02_Pin
- added J16: 220IN, Connector_JST:JST_NV_B02P-NV_1x02_P5.00mm_Vertical, symbol Connector:Conn_01x02_Pin
- RV1: value S10K460 -> CNR-07D431K; footprint Varistor:RV_Disc_D12mm_W7.9mm_P7.5mm -> Varistor:RV_Disc_D9mm_W5.2mm_P5mm
Connections:
- net L: now also J16.1 (Pin_1)
- net N: now also J16.2 (Pin_2)
