File: HVAC/UnderfloorHeating/UnderfloorHeatingActuatorsControl/220V/uhc-12/uhc-12.kicad_sch (KiCad schematic)
At the start: 21 parts, among them J1 JTAG, J1.1 EXT1.1, J1.2 EXT1.2, J10 A9, J11 A10, J12 A11, J13 A12, J14 220IN, J2 A1, J3 A2, J4 A3, J5 A4, J6 A5, J7 A6, J8 A7, J9 A8

Commit message: Reorganization
Parts:
- removed C1: TAJA105K025RNJ, Capacitor_Tantalum_SMD_AKL:CP_EIA-3216-18_Kemet-A, symbol Capacitor_AKL:CP_SMD_Tantalum_Kemet-A_3216
- removed D1: ESDA5V3SC5, Package_TO_SOT_SMD_AKL:SOT-23-5, symbol PCM_Diode_TVS_AKL:ESDA5V3SC5
- removed F1: 2A/250V/FH-1096, Fuse:Fuseholder_Clip-5x20mm_Bel_FC-203-22_Lateral_P17.80x5.00mm_D1.17mm_Horizontal, symbol Device:Fuse
- removed J1.1: EXT1.1, Connector_PinHeader_2.54mm:PinHeader_1x19_P2.54mm_Vertical, symbol Connector:Conn_01x19_Socket
- removed J1.2: EXT1.2, Connector_PinHeader_2.54mm:PinHeader_1x19_P2.54mm_Vertical, symbol Connector:Conn_01x19_Socket
- removed PS1: ZP05S0500WB, My Footprints:ZP05SXX00WB, symbol Converter_ACDC:HLK-5M03
- removed RV1: S10K460, Varistor:RV_Disc_D12mm_W7.9mm_P7.5mm, symbol Device:Varistor
- added J1: RS-232, Connector:Tag-Connect_TC2030-IDC-NL_2x03_P1.27mm_Vertical, symbol Connector:Conn_01x06_Pin
- added U1: ESP32-WROOM-32, RF_Module:ESP32-WROOM-32, symbol RF_Module:ESP32-WROOM-32
- renumbered J9 to J10, J10 to J11, J11 to J12, J12 to J13, J13 to J14, J14 to J15, J2 to J3, J3 to J4, J4 to J5, J5 to J6, J6 to J7, J7 to J8, J8 to J9
Connections:
- net +3.3V: now also U1.2 (VDD)
- net ESP_EN: now also U1.3 (EN)
- net GPI34: now also U1.6 (IO34)
- net GPI35: now also U1.7 (IO35)
- net GPI36: now also U1.4 (SENSOR_VP)
- net GPI39: now also U1.5 (SENSOR_VN)
- net GPIO0: now also U1.25 (IO0)
- net GPIO1: now also U1.35 (TXD0/IO1)
- net GPIO12: now also U1.14 (IO12)
- net GPIO13: now also U1.16 (IO13)
- net GPIO14: now also U1.13 (IO14)
- net GPIO15: now also U1.23 (IO15)
- net GPIO16: now also U1.27 (IO16)
- net GPIO17: now also U1.28 (IO17)
- net GPIO18: now also U1.30 (IO18)
- net GPIO19: now also U1.31 (IO19)
- net GPIO2: now also U1.24 (IO2)
- net GPIO21: now also U1.33 (IO21)
- net GPIO22: now also U1.36 (IO22)
- net GPIO23: now also U1.37 (IO23)
- net GPIO25: now also U1.10 (IO25)
- net GPIO26: now also U1.11 (IO26)
- net GPIO27: now also U1.12 (IO27)
- net GPIO3: now also U1.34 (RXD0/IO3)
- net GPIO32: now also U1.8 (IO32)
- net GPIO33: now also U1.9 (IO33)
- net GPIO4: now also U1.26 (IO4)
- net GPIO5: now also U1.29 (IO5)
- net GNDREF renamed GND
- net GND: now also U1.1 (GND), U1.15 (GND), U1.38 (GND), U1.39 (GND)
- new net GPIO01: J1.3 (Pin_3)
- new net GPIO03: J1.4 (Pin_4)
- new net Power/+5V_USB: J1.1 (Pin_1)
Other:
- added sheet Power (power_sch.kicad_sch)
