File: HVAC/UnderfloorHeating/UnderfloorHeatingActuatorsControl/220V/uhc-4/uhc-4.kicad_sch (KiCad schematic)
At the start: 7 parts, among them J1 JTAG, J1 RS-232, J2 Out1, J2 Out2, J2 Out3, J2 Out4, U1 ESP32-WROOM-32

Commit message: Reorganization
Parts:
- removed J1: JTAG, Connector:Tag-Connect_TC2050-IDC-FP_2x05_P1.27mm_Vertical, symbol Connector_Generic:Conn_02x05_Counter_Clockwise
- removed J2: Out1, Connector_JST:JST_NV_B02P-NV_1x02_P5.00mm_Vertical, symbol Connector:Conn_01x02_Pin
- removed J2: Out4, Connector_JST:JST_NV_B02P-NV_1x02_P5.00mm_Vertical, symbol Connector:Conn_01x02_Pin
- removed J2: Out3, Connector_JST:JST_NV_B02P-NV_1x02_P5.00mm_Vertical, symbol Connector:Conn_01x02_Pin
- removed J2: Out2, Connector_JST:JST_NV_B02P-NV_1x02_P5.00mm_Vertical, symbol Connector:Conn_01x02_Pin
- added H1, H2: MountingHole, MountingHole:MountingHole_2.7mm_M2.5_ISO7380, symbol Mechanical:MountingHole
- added R4: 470k, Resistor_SMD:R_0805_2012Metric, symbol Device:R
- U4: renamed from U1; footprint RF_Module:ESP32-WROOM-32 -> My Footprints:ESP32-WROOM-32-0.3-via
Connections:
- net ESP_EN: now also R4.2
- net GND: now also J1.5 (Pin_5)
- net Power/3V3 renamed +3V3
- net +3V3: now also R4.1
Other:
- sheet PowerOut ports: added none; removed 220V_out, 220_IN
- sheet PowerOut1 ports: added none; removed 220V_out, 220_IN
- sheet PowerOut2 ports: added none; removed 220V_out, 220_IN
- sheet PowerOut3 ports: added none; removed 220V_out, 220_IN
- company: (none) -> Wildsystems LTD
- title: (none) -> Optotriac output
