File: HVAC/UnderfloorHeating/UnderfloorHeatingActuatorsControl/24v/uhc-24-8/power.kicad_sch (KiCad schematic)
At the start: 14 parts, among them U2 LM3671MFX-3.3/NOPB

Commit message: For review
Parts:
- added D2: BAT46W, Diode_SMD:D_SOD-123, symbol Device:D_Schottky
- C2: footprint Capacitor_THT:CP_Radial_D12.5mm_P5.00mm -> Capacitor_THT_AKL:C_Radial_D4.0mm_H5.0mm_P1.50mm
- C3: footprint Capacitor_THT:CP_Radial_D12.5mm_P5.00mm -> Capacitor_THT:C_Radial_D5.0mm_H11.0mm_P2.00mm
- C5: footprint Capacitor_THT:CP_Radial_D12.5mm_P5.00mm -> Capacitor_THT:C_Radial_D4.0mm_H7.0mm_P1.50mm
- D1: footprint Diode_SMD_AKL:D_SOD-123 -> Diode_SMD_AKL:D_SOD-323
Connections:
- net GND: now also D2.2 (A)
- net at F1.2, L1.1, RV1.1: now also D2.1 (K)
Changed lines of the file:
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@@
   (junction (at 217.17 33.655) (diameter 0) (color 0 0 0 0)
   )
+  (junction (at 48.895 69.85) (diameter 0) (color 0 0 0 0)
+  )
   (junction (at 220.98 33.655) (diameter 0) (color 0 0 0 0)
   )
+  (junction (at 48.895 92.71) (diameter 0) (color 0 0 0 0)
+  )
   (junction (at 207.645 85.09) (diameter 0) (color 0 0 0 0)
   )
@@
     (stroke (width 0) (type default))
   )
-  (wire (pts (xy 37.465 92.71) (xy 53.975 92.71))
+  (wire (pts (xy 37.465 92.71) (xy 48.895 92.71))
+    (stroke (width 0) (type default))
+  )
+  (wire (pts (xy 48.895 92.71) (xy 53.975 92.71))
     (stroke (width 0) (type default))
   )
@@
     (stroke (width 0) (type default))
   )
-  (wire (pts (xy 45.085 69.85) (xy 53.975 69.85))
+  (wire (pts (xy 45.085 69.85) (xy 48.895 69.85))
     (stroke (width 0) (type default))
   )
@@
     (stroke (width 0) (type default))
   )
+  (wire (pts (xy 48.895 82.55) (xy 48.895 92.71))
+    (stroke (width 0) (type default))
+  )
   (wire (pts (xy 182.88 33.655) (xy 186.69 33.655))
     (stroke (width 0) (type default))
@@
     (stroke (width 0) (type default))
   )
+  (wire (pts (xy 48.895 69.85) (xy 53.975 69.85))
+    (stroke (width 0) (type default))
+  )
   (wire (pts (xy 149.86 74.93) (xy 161.925 74.93))
+    (stroke (width 0) (type default))
+  )
+  (wire (pts (xy 48.895 69.85) (xy 48.895 74.93))
     (stroke (width 0) (type default))
   )
@@
     (pin "1")
     (instances
-      (project "untitled"
+      (project "uhc-24-8"
         (path "/478d7b68-a2c6-4f38-9145-a627e6259a83/6e46bb13-2a97-4ee7-a91d-380b85784294"
           (reference "F1") (unit 1)
@@
     (pin "2")
     (instances
-      (project "untitled"
+      (project "uhc-24-8"
         (path "/478d7b68-a2c6-4f38-9145-a627e6259a83/6e46bb13-2a97-4ee7-a91d-380b85784294"
           (reference "C1") (unit 1)
@@
     )
   )
+  (symbol (lib_id "Device:D_Schottky") (at 48.895 78.74 270) (unit 1)
+    (in_bom yes) (on_board yes) (dnp no)
+    (property "Reference" "D2" (at 42.545 76.835 90)
+      (effects (font (size 1.27 1.27)) (justify left))
+    )
+    (property "Value" "BAT46W" (at 38.1 81.28 90)
+      (effects (font (size 1.27 1.27)) (justify left))
+    )
+    (property "Footprint" "Diode_SMD:D_SOD-123" (at 48.895 78.74 0)
+      (effects (font (size 1.27 1.27)) hide)
+    )
+    (property "Datasheet" "~" (at 48.895 78.74 0)
+      (effects (font (size 1.27 1.27)) hide)
+    )
+    (pin "1")
+    (pin "2")
+    (instances
+      (project "uhc-24-8"
+        (path "/478d7b68-a2c6-4f38-9145-a627e6259a83/6e46bb13-2a97-4ee7-a91d-380b85784294"
+          (reference "D2") (unit 1)
+        )
+      )
+    )
+  )
   (symbol (lib_id "Capacitor_AKL:C_0805") (at 174.625 37.465 0) (unit 1)
     (in_bom yes) (on_board yes) (dnp no) (fields_autoplaced)
@@
     (pin "2")
     (instances
-      (project "untitled"
+      (project "uhc-24-8"
         (path "/478d7b68-a2c6-4f38-9145-a627e6259a83/6e46bb13-2a97-4ee7-a91d-380b85784294"
           (reference "C4") (unit 1)
@@
       (effects (font (size 1.27 1.27)) (justify left))
     )
-    (property "Footprint" "Capacitor_THT:CP_Radial_D12.5mm_P5.00mm" (at 129.8702 81.28 0)
+    (property "Footprint" "Capacitor_THT:C_Radial_D5.0mm_H11.0mm_P2.00mm" (at 129.8702 81.28 0)
       (effects (font (size 1.27 1.27)) hide)
     )
@@
     (pin "2")
     (instances
-      (project "untitled"
+      (project "uhc-24-8"
         (path "/478d7b68-a2c6-4f38-9145-a627e6259a83/6e46bb13-2a97-4ee7-a91d-380b85784294"
           (reference "C3") (unit 1)
@@
     (pin "1")
     (instances
-      (project "untitled"
+      (project "uhc-24-8"
         (path "/478d7b68-a2c6-4f38-9145-a627e6259a83/6e46bb13-2a97-4ee7-a91d-380b85784294"
           (reference "#PWR08") (unit 1)
@@
     (pin "1")
     (instances
-      (project "untitled"
+      (project "uhc-24-8"
         (path "/478d7b68-a2c6-4f38-9145-a627e6259a83/6e46bb13-2a97-4ee7-a91d-380b85784294"
           (reference "#PWR09") (unit 1)
@@
     (pin "1")
     (instances
-      (project "untitled"
+      (project "uhc-24-8"
         (path "/478d7b68-a2c6-4f38-9145-a627e6259a83/6e46bb13-2a97-4ee7-a91d-380b85784294"
           (reference "#FLG03") (unit 1)
@@
       (effects (font (size 1.27 1.27)) (justify left))
     )
-    (property "Footprint" "Capacitor_THT:CP_Radial_D12.5mm_P5.00mm" (at 214.9602 83.82 0)
+    (property "Footprint" "Capacitor_THT:C_Radial_D4.0mm_H7.0mm_P1.50mm" (at 214.9602 83.82 0)
       (effects (font (size 1.27 1.27)) hide)
     )
@@
     (pin "2")
     (instances
-      (project "untitled"
+      (project "uhc-24-8"
         (path "/478d7b68-a2c6-4f38-9145-a627e6259a83/6e46bb13-2a97-4ee7-a91d-380b85784294"
           (reference "C5") (unit 1)
@@
     (pin "1")
     (instances
-      (project "untitled"
+      (project "uhc-24-8"
         (path "/478d7b68-a2c6-4f38-9145-a627e6259a83/6e46bb13-2a97-4ee7-a91d-380b85784294"
           (reference "L3") (unit 1)
@@
     (pin "2")
     (instances
-      (project "untitled"
+      (project "uhc-24-8"
         (path "/478d7b68-a2c6-4f38-9145-a627e6259a83/6e46bb13-2a97-4ee7-a91d-380b85784294"
           (reference "RV1") (unit 1)
@@
     (pin "1")
     (instances
-      (project "untitled"
+      (project "uhc-24-8"
         (path "/478d7b68-a2c6-4f38-9145-a627e6259a83/6e46bb13-2a97-4ee7-a91d-380b85784294"
           (reference "L2") (unit 1)
@@
     (pin "1")
     (instances
-      (project "untitled"
+      (project "uhc-24-8"
         (path "/478d7b68-a2c6-4f38-9145-a627e6259a83/6e46bb13-2a97-4ee7-a91d-380b85784294"
           (reference "#PWR07") (unit 1)
@@
     (pin "2")
     (instances
-      (project "untitled"
+      (project "uhc-24-8"
         (path "/478d7b68-a2c6-4f38-9145-a627e6259a83/6e46bb13-2a97-4ee7-a91d-380b85784294"
           (reference "C6") (unit 1)
@@
       (effects (font (size 1.27 1.27)) (justify left))
     )
-    (property "Footprint" "Capacitor_THT:CP_Radial_D12.5mm_P5.00mm" (at 100.0252 81.915 0)
+    (property "Footprint" "Capacitor_THT_AKL:C_Radial_D4.0mm_H5.0mm_P1.50mm" (at 100.0252 81.915 0)
       (effects (font (size 1.27 1.27)) hide)
     )
@@
     (pin "2")
     (instances
-      (project "untitled"
+      (project "uhc-24-8"
         (path "/478d7b68-a2c6-4f38-9145-a627e6259a83/6e46bb13-2a97-4ee7-a91d-380b85784294"
           (reference "C2") (unit 1)
@@
       (effects (font (size 1.27 1.27)))
     )
-    (property "Footprint" "Diode_SMD_AKL:D_SOD-123" (at 161.29 29.21 0)
+    (property "Footprint" "Diode_SMD_AKL:D_SOD-323" (at 161.29 29.21 0)
       (effects (font (size 1.27 1.27)) hide)
     )
@@
     (pin "1")
     (instances
-      (project "untitled"
+      (project "uhc-24-8"
         (path "/478d7b68-a2c6-4f38-9145-a627e6259a83/6e46bb13-2a97-4ee7-a91d-380b85784294"
           (reference "D1") (unit 1)
@@
     (pin "1")
     (instances
-      (project "untitled"
+      (project "uhc-24-8"
         (path "/478d7b68-a2c6-4f38-9145-a627e6259a83/6e46bb13-2a97-4ee7-a91d-380b85784294"
           (reference "L1") (unit 1)
@@
     (pin "1")
     (instances
-      (project "untitled"
+      (project "uhc-24-8"
         (path "/478d7b68-a2c6-4f38-9145-a627e6259a83/6e46bb13-2a97-4ee7-a91d-380b85784294"
           (reference "#PWR06") (unit 1)
@@
     (pin "1")
     (instances
-      (project "untitled"
+      (project "uhc-24-8"
         (path "/478d7b68-a2c6-4f38-9145-a627e6259a83/6e46bb13-2a97-4ee7-a91d-380b85784294"
           (reference "PS1") (unit 1)
@@
     (pin "5")
     (instances
-      (project "untitled"
+      (project "uhc-24-8"
         (path "/478d7b68-a2c6-4f38-9145-a627e6259a83/6e46bb13-2a97-4ee7-a91d-380b85784294"
           (reference "U2") (unit 1)
