File: HVAC/UnderfloorHeating/UnderfloorHeatingActuatorsControl/24v/uhc-24-8/uhc-24-8.kicad_pcb (KiCad board)
At the start: 2 copper layers, 118.1 x 69.8 mm, 56 parts, among them J1 WJ126V-5.0-2P, J10 WJ126V-5.0-2P, J11 WJ126V-5.0-2P, J2 ESP-PROG, J3 Conn_02x06_Counter_Clockwise, J4 WJ126V-5.0-2P, J5 WJ126V-5.0-2P, J6 WJ126V-5.0-2P, J7 WJ126V-5.0-2P, J8 WJ126V-5.0-2P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

Commit message: For review
Parts:
- added D2: BAT46W, Diode_SMD:D_SOD-123, F.Cu at (44.7, 107.4)
- C2: footprint Capacitor_THT:CP_Radial_D12.5mm_P5.00mm -> Capacitor_THT_AKL:C_Radial_D4.0mm_H5.0mm_P1.50mm
- C3: footprint Capacitor_THT:CP_Radial_D12.5mm_P5.00mm -> Capacitor_THT:C_Radial_D5.0mm_H11.0mm_P2.00mm
- C5: footprint Capacitor_THT:CP_Radial_D12.5mm_P5.00mm -> Capacitor_THT:C_Radial_D4.0mm_H7.0mm_P1.50mm
- D1: footprint Diode_SMD_AKL:D_SOD-123 -> Diode_SMD_AKL:D_SOD-323
- H1, H2, H3, H4: footprint MountingHole:MountingHole_6.4mm_M6 -> MountingHole:MountingHole_3.2mm_M3
Routing:
- net GND: track 10.7 -> 3.43 mm
- net Net-(D2-K): track 16.9 -> 22.0 mm
- net Net-(C1-Pad1): track 30.4 -> 29.7 mm
- net Net-(D1-K): track 73.3 -> 73.8 mm
