File: HVAC/UnderfloorHeating/UnderfloorHeatingActuatorsControl/24v/uhc-24-8/uhc-24-8.kicad_sch (KiCad schematic)
At the start: 9 parts, among them J1 WJ126V-5.0-2P, J2 ESP-PROG, J3 Conn_02x06_Counter_Clockwise, U1 ESP32-WROOM-32D

Commit message: For review
Parts:
- H1, H2, H3, H4, J3: now not fitted; now left out of the parts list
Changed lines of the file:
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@@
     (pin "2")
     (instances
-      (project "untitled"
+      (project "uhc-24-8"
         (path "/478d7b68-a2c6-4f38-9145-a627e6259a83"
           (reference "R1") (unit 1)
@@
     )
   )
-  (symbol (lib_id "Mechanical:MountingHole") (at 186.055 136.525 0) (unit 1)
-    (in_bom yes) (on_board yes) (dnp no) (fields_autoplaced)
-    (property "Reference" "H1" (at 188.595 135.3129 0)
-      (effects (font (size 1.27 1.27)) (justify left))
-    )
-    (property "Value" "MountingHole" (at 188.595 137.7371 0)
-      (effects (font (size 1.27 1.27)) (justify left))
-    )
-    (property "Footprint" "MountingHole:MountingHole_3.2mm_M3" (at 186.055 136.525 0)
-      (effects (font (size 1.27 1.27)) hide)
-    )
-    (property "Datasheet" "~" (at 186.055 136.525 0)
-      (effects (font (size 1.27 1.27)) hide)
-    )
-    (instances
-      (project "untitled"
+  (symbol (lib_id "Mechanical:MountingHole") (at 179.705 148.59 0) (unit 1)
+    (in_bom no) (on_board yes) (dnp yes) (fields_autoplaced)
+    (property "Reference" "H1" (at 182.245 147.3779 0)
+      (effects (font (size 1.27 1.27)) (justify left))
+    )
+    (property "Value" "MountingHole" (at 182.245 149.8021 0)
+      (effects (font (size 1.27 1.27)) (justify left))
+    )
+    (property "Footprint" "MountingHole:MountingHole_3.2mm_M3" (at 179.705 148.59 0)
+      (effects (font (size 1.27 1.27)) hide)
+    )
+    (property "Datasheet" "~" (at 179.705 148.59 0)
+      (effects (font (size 1.27 1.27)) hide)
+    )
+    (instances
+      (project "uhc-24-8"
         (path "/478d7b68-a2c6-4f38-9145-a627e6259a83"
           (reference "H1") (unit 1)
@@
   )
   (symbol (lib_id "Connector_Generic:Conn_02x06_Counter_Clockwise") (at 200.66 116.84 0) (unit 1)
-    (in_bom yes) (on_board yes) (dnp no) (fields_autoplaced)
+    (in_bom no) (on_board yes) (dnp yes) (fields_autoplaced)
     (property "Reference" "J3" (at 201.93 106.3457 0)
       (effects (font (size 1.27 1.27)))
@@
     )
     (property "Datasheet" "~" (at 200.66 116.84 0)
+      (effects (font (size 1.27 1.27)) hide)
+    )
+    (property "Sim.Enable" "0" (at 200.66 116.84 0)
       (effects (font (size 1.27 1.27)) hide)
     )
@@
     (pin "10")
     (instances
-      (project "untitled"
+      (project "uhc-24-8"
         (path "/478d7b68-a2c6-4f38-9145-a627e6259a83"
           (reference "J3") (unit 1)
@@
     (pin "28")
     (instances
-      (project "untitled"
+      (project "uhc-24-8"
         (path "/478d7b68-a2c6-4f38-9145-a627e6259a83"
           (reference "U1") (unit 1)
@@
     (pin "1")
     (instances
-      (project "untitled"
+      (project "uhc-24-8"
         (path "/478d7b68-a2c6-4f38-9145-a627e6259a83"
           (reference "#PWR05") (unit 1)
@@
     (pin "1")
     (instances
-      (project "untitled"
+      (project "uhc-24-8"
         (path "/478d7b68-a2c6-4f38-9145-a627e6259a83"
           (reference "J2") (unit 1)
@@
     (pin "1")
     (instances
-      (project "untitled"
+      (project "uhc-24-8"
         (path "/478d7b68-a2c6-4f38-9145-a627e6259a83"
           (reference "#PWR01") (unit 1)
@@
     (pin "1")
     (instances
-      (project "untitled"
+      (project "uhc-24-8"
         (path "/478d7b68-a2c6-4f38-9145-a627e6259a83"
           (reference "#FLG01") (unit 1)
@@
     (pin "2")
     (instances
-      (project "untitled"
+      (project "uhc-24-8"
         (path "/478d7b68-a2c6-4f38-9145-a627e6259a83"
           (reference "J1") (unit 1)
@@
     (pin "1")
     (instances
-      (project "untitled"
+      (project "uhc-24-8"
         (path "/478d7b68-a2c6-4f38-9145-a627e6259a83"
           (reference "#PWR02") (unit 1)
@@
     )
   )
-  (symbol (lib_id "Mechanical:MountingHole") (at 209.55 144.78 0) (unit 1)
-    (in_bom yes) (on_board yes) (dnp no) (fields_autoplaced)
-    (property "Reference" "H4" (at 212.09 143.5679 0)
-      (effects (font (size 1.27 1.27)) (justify left))
-    )
-    (property "Value" "MountingHole" (at 212.09 145.9921 0)
-      (effects (font (size 1.27 1.27)) (justify left))
-    )
-    (property "Footprint" "MountingHole:MountingHole_3.2mm_M3" (at 209.55 144.78 0)
-      (effects (font (size 1.27 1.27)) hide)
-    )
-    (property "Datasheet" "~" (at 209.55 144.78 0)
-      (effects (font (size 1.27 1.27)) hide)
-    )
-    (instances
-      (project "untitled"
+  (symbol (lib_id "Mechanical:MountingHole") (at 203.2 156.845 0) (unit 1)
+    (in_bom no) (on_board yes) (dnp yes) (fields_autoplaced)
+    (property "Reference" "H4" (at 205.74 155.6329 0)
+      (effects (font (size 1.27 1.27)) (justify left))
+    )
+    (property "Value" "MountingHole" (at 205.74 158.0571 0)
+      (effects (font (size 1.27 1.27)) (justify left))
+    )
+    (property "Footprint" "MountingHole:MountingHole_3.2mm_M3" (at 203.2 156.845 0)
+      (effects (font (size 1.27 1.27)) hide)
+    )
+    (property "Datasheet" "~" (at 203.2 156.845 0)
+      (effects (font (size 1.27 1.27)) hide)
+    )
+    (instances
+      (project "uhc-24-8"
         (path "/478d7b68-a2c6-4f38-9145-a627e6259a83"
           (reference "H4") (unit 1)
@@
     )
   )
-  (symbol (lib_id "Mechanical:MountingHole") (at 209.55 137.16 0) (unit 1)
-    (in_bom yes) (on_board yes) (dnp no) (fields_autoplaced)
-    (property "Reference" "H3" (at 212.09 135.9479 0)
-      (effects (font (size 1.27 1.27)) (justify left))
-    )
-    (property "Value" "MountingHole" (at 212.09 138.3721 0)
-      (effects (font (size 1.27 1.27)) (justify left))
-    )
-    (property "Footprint" "MountingHole:MountingHole_3.2mm_M3" (at 209.55 137.16 0)
-      (effects (font (size 1.27 1.27)) hide)
-    )
-    (property "Datasheet" "~" (at 209.55 137.16 0)
-      (effects (font (size 1.27 1.27)) hide)
-    )
-    (instances
-      (project "untitled"
+  (symbol (lib_id "Mechanical:MountingHole") (at 203.2 149.225 0) (unit 1)
+    (in_bom no) (on_board yes) (dnp yes) (fields_autoplaced)
+    (property "Reference" "H3" (at 205.74 148.0129 0)
+      (effects (font (size 1.27 1.27)) (justify left))
+    )
+    (property "Value" "MountingHole" (at 205.74 150.4371 0)
+      (effects (font (size 1.27 1.27)) (justify left))
+    )
+    (property "Footprint" "MountingHole:MountingHole_3.2mm_M3" (at 203.2 149.225 0)
+      (effects (font (size 1.27 1.27)) hide)
+    )
+    (property "Datasheet" "~" (at 203.2 149.225 0)
+      (effects (font (size 1.27 1.27)) hide)
+    )
+    (instances
+      (project "uhc-24-8"
         (path "/478d7b68-a2c6-4f38-9145-a627e6259a83"
           (reference "H3") (unit 1)
@@
     )
   )
-  (symbol (lib_id "Mechanical:MountingHole") (at 186.055 144.145 0) (unit 1)
-    (in_bom yes) (on_board yes) (dnp no) (fields_autoplaced)
-    (property "Reference" "H2" (at 188.595 142.9329 0)
-      (effects (font (size 1.27 1.27)) (justify left))
-    )
-    (property "Value" "MountingHole" (at 188.595 145.3571 0)
-      (effects (font (size 1.27 1.27)) (justify left))
-    )
-    (property "Footprint" "MountingHole:MountingHole_3.2mm_M3" (at 186.055 144.145 0)
-      (effects (font (size 1.27 1.27)) hide)
-    )
-    (property "Datasheet" "~" (at 186.055 144.145 0)
-      (effects (font (size 1.27 1.27)) hide)
-    )
-    (instances
-      (project "untitled"
+  (symbol (lib_id "Mechanical:MountingHole") (at 179.705 156.21 0) (unit 1)
+    (in_bom no) (on_board yes) (dnp yes) (fields_autoplaced)
+    (property "Reference" "H2" (at 182.245 154.9979 0)
+      (effects (font (size 1.27 1.27)) (justify left))
+    )
+    (property "Value" "MountingHole" (at 182.245 157.4221 0)
+      (effects (font (size 1.27 1.27)) (justify left))
+    )
+    (property "Footprint" "MountingHole:MountingHole_3.2mm_M3" (at 179.705 156.21 0)
+      (effects (font (size 1.27 1.27)) hide)
+    )
+    (property "Datasheet" "~" (at 179.705 156.21 0)
+      (effects (font (size 1.27 1.27)) hide)
+    )
+    (instances
+      (project "uhc-24-8"
         (path "/478d7b68-a2c6-4f38-9145-a627e6259a83"
           (reference "H2") (unit 1)
@@
     (pin "1")
     (instances
-      (project "untitled"
+      (project "uhc-24-8"
         (path "/478d7b68-a2c6-4f38-9145-a627e6259a83"
           (reference "#PWR03") (unit 1)
@@
     )
     (instances
-      (project "untitled"
+      (project "uhc-24-8"
         (path "/478d7b68-a2c6-4f38-9145-a627e6259a83" (page "9"))
       )
@@
     )
     (instances
-      (project "untitled"
+      (project "uhc-24-8"
         (path "/478d7b68-a2c6-4f38-9145-a627e6259a83" (page "5"))
       )
@@
     )
     (instances
-      (project "untitled"
+      (project "uhc-24-8"
         (path "/478d7b68-a2c6-4f38-9145-a627e6259a83" (page "6"))
       )
@@
     )
     (instances
-      (project "untitled"
+      (project "uhc-24-8"
         (path "/478d7b68-a2c6-4f38-9145-a627e6259a83" (page "8"))
       )
@@
     )
     (instances
-      (project "untitled"
+      (project "uhc-24-8"
         (path "/478d7b68-a2c6-4f38-9145-a627e6259a83" (page "2"))
       )
@@
     )
     (instances
-      (project "untitled"
+      (project "uhc-24-8"
         (path "/478d7b68-a2c6-4f38-9145-a627e6259a83" (page "7"))
       )
@@
     )
     (instances
-      (project "untitled"
+      (project "uhc-24-8"
         (path "/478d7b68-a2c6-4f38-9145-a627e6259a83" (page "4"))
       )
@@
     )
     (instances
-      (project "untitled"
+      (project "uhc-24-8"
         (path "/478d7b68-a2c6-4f38-9145-a627e6259a83" (page "3"))
       )
@@
     )
     (instances
-      (project "untitled"
+      (project "uhc-24-8"
         (path "/478d7b68-a2c6-4f38-9145-a627e6259a83" (page "10"))
       )
