File: HVAC/UnderfloorHeating/UnderfloorHeatingActuatorsControl/24v/uhc-24-8/hardware/PCB/outputs.kicad_sch (KiCad schematic)
At the start: 5 parts, among them Q2 2N7002P

Commit message: Ready for fabrication
Parts:
- added D18: 1N4148W, PCM_Diode_SMD_AKL:D_SOD-123, symbol Diode_AKL:1N4148W
- added J6: WJ126V-5.0-3P, My Footprints:CONN-TH_3P-P5.08_DIBO_DB142V-5.08-3P, symbol Connector:Conn_01x03_Pin
- added K7: BSC-SS-124L, My Footprints:Relay_SPDT_QLRELAY_BSC, symbol Relay:TIANBO-HJR-4102-L
- D8: renamed from D5; LCSC Part # (none) -> C2296
- Q7: renamed from Q2; LCSC Part # (none) -> C81488
- R24: renamed from R13; LCSC Part # (none) -> C17734
- R28: renamed from R9; LCSC Part # (none) -> C17673
- R29: renamed from R8; value 56 -> 56R; LCSC Part # (none) -> C17757
Connections:
- net ACT: no longer names the net of Q7.3 (D)
- net ACT: now also D18.2 (A), K7.8
- new net +24V_FUSED: D18.1 (K), K7.5
- new net COM: J6.2 (Pin_2), K7.12
- new net NC: J6.1 (Pin_1), K7.7
- new net NO: J6.3 (Pin_3), K7.6
