File: HVAC/UnderfloorHeating/UnderfloorHeatingActuatorsControl/24v/uhc-24-8/hardware/PCB/power.kicad_sch (KiCad schematic)
At the start: 19 parts, among them U3 LM3671MFX-3.3/NOPB

Commit message: Ready for fabrication
Parts:
- removed D4: KT-0805G, LED_SMD:LED_0805_2012Metric, symbol Device:LED_Small
- removed PS1: K7805JT-500R3-LB, K7805JT-500R3:CONV_K7805JT-500R3-LB, symbol K7805JT-500R3:K7805JT-500R3-LB
- removed R7: 20, Resistor_SMD:R_0805_2012Metric, symbol Device:R
- added D28: KT-0805G, LED_SMD:LED_0805_2012Metric, symbol Device:LED_Small
- added R44: 20R, Resistor_SMD:R_0805_2012Metric, symbol Device:R
- added TP2: 5V_USB, TestPoint:TestPoint_Pad_D2.0mm, symbol Connector:TestPoint
- added TP3: 5V, TestPoint:TestPoint_Pad_D2.0mm, symbol Connector:TestPoint
- added TP4: 3.3V, TestPoint:TestPoint_Pad_D2.0mm, symbol Connector:TestPoint
- added U1: K7805-500R3, My Footprints:PWRM-TH_K78XX-500R3, symbol PCM_Voltage_Regulator_AKL:LM7805CT
- C3: renamed from C5; footprint Capacitor_THT:CP_Radial_D12.5mm_P5.00mm -> My Footprints:CAP-SMD_BD12.5-L13.0-W13.0-LS14.4-FD; LCSC Part # (none) -> C487372
- C4: renamed from C6; value 4.7uF/50V -> 4.7uF/63V; footprint Capacitor_THT_AKL:C_Radial_D4.0mm_H5.0mm_P1.50mm -> Capacitor_SMD_AKL:C_1206_3216Metric; LCSC Part # (none) -> C29823
- C5: renamed from C7; footprint Capacitor_THT:C_Radial_D5.0mm_H11.0mm_P2.00mm -> Capacitor_SMD_AKL:C_1206_3216Metric; LCSC Part # (none) -> C13585
- C6: renamed from C9; footprint Capacitor_THT:C_Radial_D4.0mm_H7.0mm_P1.50mm -> Capacitor_SMD:C_1206_3216Metric; LCSC Part # (none) -> C5672
- C7: renamed from C8; value 4.7uF -> 4.7uF/10V; footprint Capacitor_SMD_AKL:C_0805_2012Metric -> Capacitor_SMD:C_0402_1005Metric; LCSC Part # (none) -> C23733
- C8: renamed from C10; footprint Capacitor_SMD_AKL:C_0805_2012Metric -> Capacitor_SMD:C_0603_1608Metric; LCSC Part # (none) -> C19702
- D25: renamed from D1; LCSC Part # (none) -> C7420332
- D27: renamed from D2; footprint Diode_SMD_AKL:D_SOD-323 -> Diode_SMD:D_SOD-123; LCSC Part # (none) -> C3033976
- D29: renamed from D3; LCSC Part # (none) -> C2297
- F1: value C3131 -> Fuse; footprint Fuse:Fuseholder_Cylinder-5x20mm_Schurter_0031_8201_Horizontal_Open -> My Footprints:FUSE-TH_L24.4-W9.4-P22.60; LCSC Part # (none) -> C717030
- L1: value BC54-820M(CD) -> FHW1210IF820JST; footprint My Footprints:BC54-820M -> Inductor_SMD:L_1210_3225Metric; LCSC Part # (none) -> C394099
- L2: value CD31 220M -> 22uH; footprint My Footprints:CD31 -> Inductor_SMD:L_0603_1608Metric; LCSC Part # (none) -> C6808015
- L3: footprint Inductor_SMD:L_0805_2012Metric -> Ferrite_SMD_AKL:Ferrite_1206_3216Metric; LCSC Part # (none) -> C139249
- R42: renamed from R6; value 20 -> 20R; LCSC Part # (none) -> C17659
- RV1: value SFI1206SV471-201A -> RL0603E024M250K; footprint Resistor_SMD:R_1206_3216Metric -> Diode_SMD_AKL:D_0603_1608Metric; LCSC Part # (none) -> LCSC Part #
- U4: renamed from U3; value LM3671MFX-3.3/NOPB -> LM3671MFX-3.3/NOPB; LCSC Part # (none) -> C477918
Connections:
- net +3V3: now also D28.2 (A), TP4.1
- net +5V_USB: now also TP2.1
- net GND: now also R44.1, U1.2
- net +24V_FUSED: now reaches D25.1 (K), F1.2, L1.1, RV1.1
- net +5V: now reaches C6.1, C7.1, D27.1 (K), D29.2 (A), U4.1 (Vin), U4.3 (EN)
- net +5V: now also TP3.1, U1.3 (OUT)
- net at C5.1, L2.2: now also U1.1 (IN)
- new net: D28.1 (K), R44.2
Other:
- moved on the sheet: C6, C7, C8, D25, D27, L3, U4
