File: HVAC/UnderfloorHeating/UnderfloorHeatingActuatorsControl/24v/uhc-24-8/hardware/PCB/uhc-24-8.kicad_sch (KiCad schematic)
At the start: 22 parts, among them J1 WJ126V-5.0-2P, J2 ESP-PROG, J3 Conn_01x06_Socket, J4 WAGO 233-212, J5 WAGO 233-212, SW1 Reset, SW2 Test, U1 ESP32-WROOM-32D, U2 MCP23017_SS

Commit message: Ready for fabrication
Parts:
- removed C4: 0.1uF, Capacitor_SMD:C_0805_2012Metric, symbol Device:C
- removed J3: Conn_01x06_Socket, Connector_JST:JST_EH_B6B-EH-A_1x06_P2.50mm_Vertical, symbol Connector:Conn_01x06_Socket
- removed J4, J5: WAGO 233-212, WAGO:CONN_233-112_WAG, symbol Connector:Conn_01x12_Pin
- removed R2, R3, R4, R5: 10K, Resistor_SMD:R_0805_2012Metric, symbol Device:R
- added C2: 0.1uF, Capacitor_SMD:C_0402_1005Metric, symbol Device:C
- added D26: KT-0805B, Diode_SMD_AKL:D_0805_2012Metric, symbol Device:LED
- added D30: KT-0805G, LED_SMD:LED_0805_2012Metric, symbol Device:LED_Small
- added R13, R14, R15, R16: 10K, PCM_Resistor_SMD_AKL:R_0603_1608Metric, symbol Device:R
- added R43: 20R, Resistor_SMD:R_0805_2012Metric, symbol Device:R
- added R45: 15R, Resistor_SMD:R_0805_2012Metric, symbol Device:R
- added TP1: 24V, TestPoint:TestPoint_Pad_D2.0mm, symbol Connector:TestPoint
- C1: footprint Capacitor_SMD:C_0805_2012Metric -> Capacitor_SMD:C_0402_1005Metric; LCSC Part # (none) -> C14445
- C10: renamed from C3; footprint Capacitor_SMD:C_0805_2012Metric -> Capacitor_SMD:C_0402_1005Metric; LCSC Part # (none) -> C541406
- C9: renamed from C2; footprint Capacitor_SMD:C_0805_2012Metric -> Capacitor_SMD:C_0603_1608Metric; LCSC Part # (none) -> C59461
- J13: renamed from J2; now not fitted; now left out of the parts list
- J14: renamed from J1; footprint My Footprints:WJ500V-5.08-2P -> My Footprints:CONN-TH_2P-P5.08_DIBO_DB142V-5.08-2P; LCSC Part # (none) -> C2898699
- R23: renamed from R1; footprint Resistor_SMD:R_0805_2012Metric -> PCM_Resistor_SMD_AKL:R_0603_1608Metric; LCSC Part # (none) -> C25804
- SW1: value Reset -> Reboot; footprint Button_Switch_SMD:SW_Push_1P1T_NO_Vertical_Wuerth_434133025816 -> My Footprints:SW-SMD_4P-L5.1-W5.1-P3.70-LS6.5-TL-2; LCSC Part # (none) -> C318884
- SW2: value Test -> Clear; footprint Button_Switch_SMD:SW_Push_1P1T_NO_Vertical_Wuerth_434133025816 -> My Footprints:SW-SMD_4P-L5.1-W5.1-P3.70-LS6.5-TL-2; LCSC Part # (none) -> C318884
- U2: LCSC Part # (none) -> C558584
- U3: renamed from U1; footprint My Footprints:ESP32-WROOM-32-0.3-via -> My Footprints:WIFI-SMD_ESP32-WROOM-32E-A; LCSC Part # (none) -> C701341
- renumbered H4 to H3, H3 to H4
Connections:
- net +24V: now also TP1.1
- net 3v3: now also R13.1
- net GND: now also C2.2, R14.2, R15.2, R16.2, R43.1, R45.2
- net IO18: now also D26.2 (A)
- net IO19: now also D30.2 (A)
- net IO27: now also C2.1
- net Out1/IN: now also U2.8 (GPB7); no longer U2.1 (GPB0)
- net Out10/IN: now also U2.23 (GPA2); no longer U2.22 (GPA1)
- net Out11/IN: now also U2.22 (GPA1); no longer U2.23 (GPA2)
- net Out12/IN: now also U2.21 (GPA0); no longer U2.24 (GPA3)
- net Out2/IN: now also U2.7 (GPB6); no longer U2.2 (GPB1)
- net Out3/IN: now also U2.6 (GPB5); no longer U2.3 (GPB2)
- net Out4/IN: now also U2.5 (GPB4); no longer U2.4 (GPB3)
- net Out5/IN: now also U2.4 (GPB3); no longer U2.5 (GPB4)
- net Out6/IN: now also U2.3 (GPB2); no longer U2.6 (GPB5)
- net Out7/IN: now also U2.1 (GPB0); no longer U2.7 (GPB6)
- net Out8/IN: now also U2.2 (GPB1); no longer U2.8 (GPB7)
- net Out9/IN: now also U2.24 (GPA3); no longer U2.21 (GPA0)
- net at U2.16 (A1): now also R15.1
- net at U2.17 (A2): now also R14.1
- net at U2.15 (A0): now also R16.1
- net at U2.18 (~{RESET}): now also R13.2
- new net: D26.1 (K), R45.1
- new net: D30.1 (K), R43.2
- no-connect marks 26 -> 23
Other:
- sheet Out1 ports: added none; removed ACT
- sheet Out10 ports: added none; removed ACT
- sheet Out11 ports: added none; removed ACT
- sheet Out12 ports: added none; removed ACT
- sheet Out2 ports: added none; removed ACT
- sheet Out3 ports: added none; removed ACT
- sheet Out4 ports: added none; removed ACT
- sheet Out5 ports: added none; removed ACT
- sheet Out6 ports: added none; removed ACT
- sheet Out7 ports: added none; removed ACT
- sheet Out8 ports: added none; removed ACT
- sheet Out9 ports: added none; removed ACT
